File: DeskPresence.kicad_sch (KiCad schematic)
At the start: 1 part, among them J1 USB_A

Commit message: Sketchy first pcb
Parts:
- added C1, C2: C_Polarized, Capacitor_THT:CP_Radial_D6.3mm_P2.50mm, symbol Device:C_Polarized
- added J2: TTL, Connector_PinHeader_2.54mm:PinHeader_1x04_P2.54mm_Vertical, symbol ftdi-connector:TTL
- added SW1: MODE, Connector_PinHeader_2.54mm:PinHeader_1x03_P2.54mm_Vertical, symbol Switch:SW_Push
- added SW2: RESET, Connector_PinHeader_2.54mm:PinHeader_1x03_P2.54mm_Vertical, symbol Switch:SW_Push
- added U1: UA78M33_TO252, Package_TO_SOT_SMD:TO-252-2, symbol Regulator_Linear:KA78M05_TO252
- added U2: esp-01m, esp-01m:esp-01m, symbol esp-01m:esp-01m
- added U3: GP2Y0A02YK0F, GP2Y0A02YK0F:GP2Y0A02YK0F, symbol GP2Y0A02YK0F:GP2Y0A02YK0F
Connections:
- net +5V: now reaches J1.1 (VBUS)
- net +5V: now also C1.1, U1.1 (VI)
- net GND: now reaches J1.4 (GND)
- net GND: now also J1.5 (Shield), C1.2, C2.2, J2.1 (GND), SW1.2, SW2.2, U1.2 (GND), U2.1 (GND), U3.1 (GND)
- new net: SW2.1, U2.18 (RST)
- new net: SW1.1, U2.8 (GP0)
- new net +3V3: C2.1, J2.4 (VDD), U1.3 (VO), U2.2 (VDD), U2.9 (EN), U3.2 (VCC)
- new net Data: U2.16 (ADC), U3.3 (VOUT)
- new net RX: J2.3 (TX), U2.4 (GP3/RX)
- new net TX: J2.2 (RX), U2.3 (GP2/TX)
- no-connect marks 0 -> 2
Other:
- company: (none) -> Besmer Labs
- title: (none) -> DeskPresence
- moved on the sheet: J1
